File: pcb/LoraHarvesterBox.kicad_sch (KiCad schematic)
At the start: 45 parts, among them J1 Conn_01x02_Pin, J2 Conn_01x02_Pin, J3 Conn_01x02_Pin, J4 Conn_01x04_Socket, J5 Conn_01x04_Socket, J6 Conn_01x04_Socket, J7 Conn_01x04_Socket, J8 Conn_01x06_Socket, J9 Conn_01x08_Socket, SW1 SSSS811101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

Commit message: docs, pcb, sch: add missing buffer capacitor to power switch
Parts:
- added C6: 1uF, Capacitor_SMD:C_0603_1608Metric_Pad1.08x0.95mm_HandSolder, symbol Device:C
Connections:
- net +3V0: now also C6.2
- net GND: now also C6.1
Changed lines of the file:
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@@
 	)
 	(junction
+		(at 87.63 199.39)
+		(diameter 0)
+		(color 0 0 0 0)
+	)
+	(junction
 		(at 154.94 114.3)
 		(diameter 0)
@@
 	(wire
 		(pts
+			(xy 87.63 199.39) (xy 106.68 199.39)
+		)
+		(stroke
+			(width 0)
+			(type default)
+		)
+	)
+	(wire
+		(pts
 			(xy 207.01 66.04) (xy 207.01 52.07)
 		)
@@
 	(wire
 		(pts
-			(xy 104.14 196.85) (xy 104.14 199.39)
-		)
-		(stroke
-			(width 0)
-			(type default)
-		)
-	)
-	(wire
-		(pts
 			(xy 173.99 133.35) (xy 173.99 137.16)
 		)
@@
 	(wire
 		(pts
+			(xy 87.63 208.28) (xy 87.63 209.55)
+		)
+		(stroke
+			(width 0)
+			(type default)
+		)
+	)
+	(wire
+		(pts
 			(xy 41.91 92.71) (xy 48.26 92.71)
 		)
@@
 	(wire
 		(pts
+			(xy 87.63 200.66) (xy 87.63 199.39)
+		)
+		(stroke
+			(width 0)
+			(type default)
+		)
+	)
+	(wire
+		(pts
 			(xy 200.66 36.83) (xy 200.66 30.48)
 		)
@@
 	(wire
 		(pts
-			(xy 104.14 199.39) (xy 106.68 199.39)
+			(xy 81.28 199.39) (xy 87.63 199.39)
 		)
 		(stroke
@@
 	)
 	(symbol
+		(lib_id "Device:C")
+		(at 87.63 204.47 180)
+		(unit 1)
+		(exclude_from_sim no)
+		(in_bom yes)
+		(on_board yes)
+		(dnp no)
+		(fields_autoplaced yes)
+		(property "Reference" "C6"
+			(at 91.44 203.1999 0)
+			(effects
+				(font
+					(size 1.27 1.27)
+				)
+				(justify right)
+			)
+		)
+		(property "Value" "1uF"
+			(at 91.44 205.7399 0)
+			(effects
+				(font
+					(size 1.27 1.27)
+				)
+				(justify right)
+			)
+		)
+		(property "Footprint" "Capacitor_SMD:C_0603_1608Metric_Pad1.08x0.95mm_HandSolder"
+			(at 86.6648 200.66 0)
+			(effects
+				(font
+					(size 1.27 1.27)
+				)
+				(hide yes)
+			)
+		)
+		(property "Datasheet" "~"
+			(at 87.63 204.47 0)
+			(effects
+				(font
+					(size 1.27 1.27)
+				)
+				(hide yes)
+			)
+		)
+		(property "Description" "Unpolarized capacitor"
+			(at 87.63 204.47 0)
+			(effects
+				(font
+					(size 1.27 1.27)
+				)
+				(hide yes)
+			)
+		)
+		(pin "2"
+		)
+		(pin "1"
+		)
+		(instances
+			(project ""
+				(path "/a6f37965-abbf-44d1-94f3-9a9b9eaa16a8"
+					(reference "C6")
+					(unit 1)
+				)
+			)
+		)
+	)
+	(symbol
 		(lib_id "power:GND")
 		(at 40.64 146.05 0)
@@
 	)
 	(symbol
+		(lib_id "power:GND")
+		(at 87.63 209.55 0)
+		(unit 1)
+		(exclude_from_sim no)
+		(in_bom yes)
+		(on_board yes)
+		(dnp no)
+		(fields_autoplaced yes)
+		(property "Reference" "#PWR040"
+			(at 87.63 215.9 0)
+			(effects
+				(font
+					(size 1.27 1.27)
+				)
+				(hide yes)
+			)
+		)
+		(property "Value" "GND"
+			(at 87.63 214.63 0)
+			(effects
+				(font
+					(size 1.27 1.27)
+				)
+			)
+		)
+		(property "Footprint" ""
+			(at 87.63 209.55 0)
+			(effects
+				(font
+					(size 1.27 1.27)
+				)
+				(hide yes)
+			)
+		)
+		(property "Datasheet" ""
+			(at 87.63 209.55 0)
+			(effects
+				(font
+					(size 1.27 1.27)
+				)
+				(hide yes)
+			)
+		)
+		(property "Description" "Power symbol creates a global label with name \"GND\" , ground"
+			(at 87.63 209.55 0)
+			(effects
+				(font
+					(size 1.27 1.27)
+				)
+				(hide yes)
+			)
+		)
+		(pin "1"
+		)
+		(instances
+			(project ""
+				(path "/a6f37965-abbf-44d1-94f3-9a9b9eaa16a8"
+					(reference "#PWR040")
+					(unit 1)
+				)
+			)
+		)
+	)
+	(symbol
 		(lib_id "Connector:Conn_01x06_Socket")
 		(at 114.3 73.66 180)
@@
 	(symbol
 		(lib_id "power:+3V0")
-		(at 104.14 196.85 0)
+		(at 81.28 199.39 90)
 		(unit 1)
 		(exclude_from_sim no)
@@
 		(fields_autoplaced yes)
 		(property "Reference" "#PWR041"
-			(at 104.14 200.66 0)
+			(at 85.09 199.39 0)
 			(effects
 				(font
@@
 		)
 		(property "Value" "+3V0"
-			(at 104.14 191.77 0)
+			(at 80.01 196.85 90)
 			(effects
 				(font
@@
 		)
 		(property "Footprint" ""
-			(at 104.14 196.85 0)
+			(at 81.28 199.39 0)
 			(effects
 				(font
@@
 		)
 		(property "Datasheet" ""
-			(at 104.14 196.85 0)
+			(at 81.28 199.39 0)
 			(effects
 				(font
@@
 		)
 		(property "Description" "Power symbol creates a global label with name \"+3V0\""
-			(at 104.14 196.85 0)
+			(at 81.28 199.39 0)
 			(effects
 				(font

Commit message: pcb, sch: load switch now controls the entire 3.3V rail
In the last version only the ST microcontroller was switched/on off by
the load switch. This caused problems with the periphery: they stayed
online with slowly fading into a brown out. This also fixes battery
drain by half-dead sensors.
Connections:
- net Vdd_Input is gone; now on net +3V0: U2.24 (VDD), U4.6 (VOUT)
- net +3V0: no longer C5.2, C6.2, L2.2, U1.14 (VOUT), U4.1 (VIN)
- net VBAT_OK: no longer U2.3 (PA15/PIN_A4)
- new net VHARVESTER: C5.2, C6.2, L2.2, U1.14 (VOUT), U4.1 (VIN)
- no-connect marks 4 -> 5
